File: Documentation/Hardware/Display - Lawo 28x24/Schematic/Lawo 28x24 Matrix Components.sch (KiCad schematic (older format))
At the start: 17 parts, among them IC1 FP2800A, IC2 FP2800A, IC3 FP2800A, P1 CONN_02X17, P2 CONN_02X17

Commit message: Lawo 28x24 Error fixed and minor layout changes
- incorrect pin at IC1-3 fixed (pin 17 was labeled as 19)
- orientation of IC1 aligned with IC2 and 3
- indicators for additional traces added (ends still unconnected)
- plotted schematics updated
Connections:
- net IC1_A0 is gone; now on net COL_A0: P1.7 (P7), P2.7 (P7)
- net IC1_A1 is gone; now on net COL_A1: P1.9 (P9), P2.9 (P9)
- net IC1_A2 is gone; now on net COL_A2: P1.11 (P11), P2.11 (P11)
- net IC1_B0 is gone; now on net COL_B0: P1.13 (P13), P2.13 (P13)
- net IC1_B1 is gone; now on net COL_B1: P1.15 (P15), P2.15 (P15)
- net +24V: now also C3.1; no longer C3.2
- net COL_ENABLE: now also C1.1; no longer C1.2
- net GND: now also C3.2, IC1.25 (GROUND), R1.2; no longer C3.1, R1.1
- new net: C1.2, IC1.24 (ENABLE), R1.1
- no-connect marks 13 -> 89
Other:
- moved on the sheet: C1, C2, C3, IC1, R1
