File: Documentation/Hardware/Display - Lawo 28x13/Schematic/Lawo 28x13 Matrix Components.sch (KiCad schematic (older format))
At the start: 7 parts, among them IC1 FP2800A, P1 CONN_02X17, P2 CONN_01X03

Commit message: Schematic for Lawo 28x13 updated for upgraded KiCad version.
- EESchema Schematic File Version 4
- KiCad 5.0.0-rc3-dev
- plots of the upgraded schematic
Parts:
- removed P1: CONN_02X17, Socket_Strips:Socket_Strip_Straight_2x17, symbol CONN_02X25
- added P1: Conn_02x25_Counter_Clockwise, Connectors_IDC:IDC-Header_2x25_Pitch2.54mm_Straight, symbol Connector:Conn_02x25_Counter_Clockwise
- C1, C2, C3: symbol C -> device:C
- IC1: symbol FP2800A -> FP2800a:FP2800A
- P2: footprint Pin_Headers:Pin_Header_Straight_1x03 -> Pin_Headers:Pin_Header_Straight_1x03_Pitch2.54mm; symbol CONN_01X03 -> Connector:Conn_01x03
- R1: symbol R -> device:R
Connections:
- wire segments 106 -> 113
Changed lines of the file:
@@
-EESchema Schematic File Version 2
-LIBS:Lawo 28x13 Matrix Components-rescue
-LIBS:power
-LIBS:device
-LIBS:transistors
-LIBS:conn
-LIBS:linear
-LIBS:regul
-LIBS:74xx
-LIBS:cmos4000
-LIBS:adc-dac
-LIBS:memory
-LIBS:xilinx
-LIBS:microcontrollers
-LIBS:dsp
-LIBS:microchip
-LIBS:analog_switches
-LIBS:motorola
-LIBS:texas
-LIBS:intel
-LIBS:audio
-LIBS:interface
-LIBS:digital-audio
-LIBS:philips
-LIBS:display
-LIBS:cypress
-LIBS:siliconi
-LIBS:opto
-LIBS:atmel
-LIBS:contrib
-LIBS:valves
-LIBS:FP2800a
-LIBS:Lawo 28x13 Matrix Components-cache
-EELAYER 25 0
+EESchema Schematic File Version 4
+EELAYER 26 0
 EELAYER END
 $Descr A4 11693 8268
@@
 Sheet 1 1
 Title "Lawo 28x13 Matrix Components"
-Date "2016-10-29"
-Rev "0.2"
+Date "2019-02-03"
+Rev "0.3"
 Comp "Flip-The-Dot"
 Comment1 "Robert Römer"
@@
 $EndDescr
 $Comp
-L VSS #PWR01
+L power:VSS #PWR01
 U 1 1 574CAF97
 P 1000 5650
@@
 $EndComp
 $Comp
-L VCC #PWR02
+L power:VCC #PWR02
 U 1 1 574CAFAE
 P 2100 5650
@@
 $EndComp
 $Comp
-L GND #PWR03
+L power:GND #PWR03
 U 1 1 574CAFC5
 P 3200 5650
@@
 $EndComp
 $Comp
-L +24V #PWR04
+L power:+24V #PWR04
 U 1 1 574CB83E
 P 1000 6800
@@
 $EndComp
 $Comp
-L +5V #PWR05
+L power:+5V #PWR05
 U 1 1 574CB85B
 P 2100 6800
@@
 $EndComp
 $Comp
-L PWR_FLAG #FLG06
+L power:PWR_FLAG #FLG06
 U 1 1 574CB8A8
 P 3250 6200
@@
 $EndComp
 $Comp
-L PWR_FLAG #FLG07
+L power:PWR_FLAG #FLG07
 U 1 1 574CB8C6
 P 2150 6200
@@
 $EndComp
 $Comp
-L PWR_FLAG #FLG08
+L power:PWR_FLAG #FLG08
 U 1 1 574CB8E7
 P 1050 6200
@@
 	1    1050 6200
 	0    1    1    0
-$EndComp
-$Comp
-L FP2800A IC1
-U 1 1 574CC9A9
-P 2550 1950
-F 0 "IC1" H 2550 2300 50  0000 C CNN
-F 1 "FP2800A" H 2550 150 50  0000 C CNN
-F 2 "Housings_DIP:DIP-40_W15.24mm_LongPads" H 2400 1950 50  0001 C CNN
-F 3 "http://pdf.datasheetcatalog.com/datasheets/320/500899_DS.pdf" H 2400 1950 50  0001 C CNN
-F 4 "Column Controller" H 2550 1950 60  0001 C CNN "Usage"
-	1    2550 1950
-	1    0    0    -1
 $EndComp
 Text GLabel 1850 3500 0    60   Input ~ 0
@@
 B1
 $Comp
-L GND #PWR09
+L power:GND #PWR09
 U 1 1 574CC9BE
 P 3900 3200
@@
 $EndComp
 $Comp
-L GND #PWR010
+L power:GND #PWR010
 U 1 1 574CC9C4
 P 1100 2300
@@
 $EndComp
 $Comp
-L VSS #PWR011
+L power:VSS #PWR011
 U 1 1 574CC9CA
 P 3900 2200
@@
 $EndComp
 $Comp
-L VCC #PWR012
+L power:VCC #PWR012
 U 1 1 574CC9D0
 P 1100 3300
@@
 DATA
 $Comp
-L R R1
+L device:R R1
 U 1 1 574E0691
 P 2100 4000
@@
 $EndComp
 $Comp
-L C C2
+L device:C C2
 U 1 1 574E0790
 P 2200 4700
@@
 $EndComp
 $Comp
-L C C1
+L device:C C1
 U 1 1 574E07E1
 P 2550 1300
@@
 $EndComp
 $Comp
-L C C3
+L device:C C3
 U 1 1 574E0815
 P 1300 3700
@@
 $EndComp
 $Comp
-L GND #PWR013
+L power:GND #PWR013
 U 1 1 574E0A70
 P 1100 4350
@@
 Power Levels
 $Comp
-L VSS #PWR014
+L power:VSS #PWR014
 U 1 1 5759D2E9
 P 4950 1500
@@
 $EndComp
 $Comp
-L GND #PWR015
+L power:GND #PWR015
 U 1 1 5759D338
 P 4750 1600
@@
 $EndComp
 $Comp
-L VCC #PWR016
+L power:VCC #PWR016
 U 1 1 5759D40F
 P 4950 1700
@@
 Text GLabel 5600 2200 0    60   Input ~ 0
 A1
-$Comp
-L CONN_02X25 P1
-U 1 1 574CBA24
-P 6350 2700
-F 0 "P1" H 6350 1350 50  0000 C CNN
-F 1 "CONN_02X17" V 6350 2700 50  0000 C CNN
-F 2 "Socket_Strips:Socket_Strip_Straight_2x17" H 6350 1600 50  0001 C CNN
-F 3 "" H 6350 1600 50  0000 C CNN
-F 4 "Socket bottom/left (Output)" H 6350 2700 60  0001 C CNN "Comment"
-F 5 "Input Connector" H 6350 2700 60  0001 C CNN "Usage"
-	1    6350 2700
-	1    0    0    -1
-$EndComp
 Text GLabel 5600 2500 0    60   BiDi ~ 0
 RESET_01
@@
 NoConn ~ 6100 2400
 $Comp
-L GND #PWR017
+L power:GND #PWR017
 U 1 1 5759D9AA
 P 4950 2300
@@
 NoConn ~ 6600 2400
 $Comp
-L GND #PWR018
+L power:GND #PWR018
 U 1 1 5759DBBC
 P 7750 2300
@@
 NoConn ~ 6600 1800
 $Comp
-L CONN_01X03 P2
+L Connector:Conn_01x03 P2
 U 1 1 5759E1D7
 P 10450 2700
 F 0 "P2" H 10450 2900 50  0000 C CNN
 F 1 "CONN_01X03" V 10550 2700 50  0000 C CNN
-F 2 "Pin_Headers:Pin_Header_Straight_1x03" H 10450 2700 50  0001 C CNN
+F 2 "Pin_Headers:Pin_Header_Straight_1x03_Pitch2.54mm" H 10450 2700 50  0001 C CNN
 F 3 "" H 10450 2700 50  0000 C CNN
 	1    10450 2700
@@
 NoConn ~ 6100 1900
 $Comp
-L VSS #PWR019
+L power:VSS #PWR019
 U 1 1 5759EE34
 P 7750 1500
@@
 $EndComp
 $Comp
-L GND #PWR020
+L power:GND #PWR020
 U 1 1 5759EE3A
 P 7950 1600
@@
 $EndComp
 $Comp
-L VCC #PWR021
+L power:VCC #PWR021
 U 1 1 5759EE40
 P 7750 1700
@@
 	3200 5650 3200 6200
 Wire Wire Line
-	2100 5650 2100 6800
-Wire Wire Line
-	1000 5650 1000 6800
+	2100 5650 2100 6200
+Wire Wire Line
+	1000 5650 1000 6200
 Wire Wire Line
 	3100 3500 3250 3500
@@
 	1850 3400 2000 3400
 Wire Wire Line
-	1100 3300 2000 3300
+	1100 3300 1300 3300
 Wire Wire Line
 	3100 3200 3900 3200
 Wire Wire Line
-	1100 2300 2000 2300
-Wire Wire Line
-	3100 2200 3900 2200
-Wire Wire Line
-	1300 4000 1950 4000
+	1100 2300 1300 2300
+Wire Wire Line
+	3100 2200 3800 2200
+Wire Wire Line
+	1300 4000 1750 4000
 Connection ~ 1750 4000
 Wire Wire Line
 	1750 4350 1100 4350
 Wire Wire Line
-	2250 4000 3800 4000
+	2250 4000 2500 4000
 Wire Wire Line
 	3800 4000 3800 3300
@@
 Wire Wire Line
 	3200 2100 3100 2100
+Wire Wire Line
+	1750 4000 1950 4000
+Wire Wire Line
+	2500 4000 3800 4000
+Wire Wire Line
+	1300 3300 2000 3300
+Wire Wire Line
+	1300 2300 2000 2300
+Wire Wire Line
+	3800 2200 3900 2200
+Wire Wire Line
+	2100 6200 2100 6800
+Wire Wire Line
+	1000 6200 1000 6800
+$Comp
+L Connector:Conn_02x25_Counter_Clockwise P1
+U 1 1 5C58080C
+P 6300 2700
+F 0 "P1" H 6350 4117 50  0000 C CNN
+F 1 "Conn_02x25_Counter_Clockwise" H 6350 4026 50  0000 C CNN
+F 2 "Connectors_IDC:IDC-Header_2x25_Pitch2.54mm_Straight" H 6300 2700 50  0001 C CNN
+F 3 "~" H 6300 2700 50  0001 C CNN
+	1    6300 2700
+	1    0    0    -1
+$EndComp
+$Comp
+L FP2800a:FP2800A IC1
+U 1 1 574CC9A9
+P 2550 1950
+F 0 "IC1" H 2550 2300 50  0000 C CNN
+F 1 "FP2800A" H 2550 150 50  0000 C CNN
+F 2 "Housings_DIP:DIP-40_W15.24mm_LongPads" H 2400 1950 50  0001 C CNN
+F 3 "http://pdf.datasheetcatalog.com/datasheets/320/500899_DS.pdf" H 2400 1950 50  0001 C CNN
+F 4 "Column Controller" H 2550 1950 60  0001 C CNN "Usage"
+	1    2550 1950
+	1    0    0    -1
+$EndComp
 $EndSCHEMATC

Commit message: Lawo 28x13 Matrix Components schematic modified to fix FP2800a wiring and labels
Connections:
- net labels added: COL_01, COL_02, COL_03, COL_04, COL_05, COL_06, COL_07, COL_08, COL_09, COL_10, COL_11, COL_12, COL_13, COL_14, COL_15, COL_16, COL_17, COL_18, COL_19, COL_20, COL_21, COL_22, COL_23, COL_24, COL_25, COL_26, COL_27, COL_28
- wire segments 113 -> 115
- no-connect marks 11 -> 9
Changed lines of the file:
@@
 EESchema Schematic File Version 4
+LIBS:Lawo 28x13 Matrix Components-cache
 EELAYER 26 0
 EELAYER END
@@
 	7750 1500 6600 1500
 Text GLabel 1900 1900 0    60   BiDi ~ 0
-RESET_13
+COL_13
 Text GLabel 1900 3200 0    60   BiDi ~ 0
-RESET_01
+COL_01
 Text GLabel 1900 3100 0    60   BiDi ~ 0
-RESET_02
+COL_02
 Text GLabel 1900 2900 0    60   BiDi ~ 0
-RESET_04
+COL_04
 Text GLabel 1900 3000 0    60   BiDi ~ 0
-RESET_03
+COL_03
 Text GLabel 1900 2700 0    60   BiDi ~ 0
-RESET_05
+COL_05
 Text GLabel 1900 2800 0    60   BiDi ~ 0
-RESET_06
+COL_06
 Text GLabel 1900 2600 0    60   BiDi ~ 0
-RESET_07
+COL_07
 Text GLabel 1900 2200 0    60   BiDi ~ 0
-RESET_08
+COL_08
 Text GLabel 1900 2100 0    60   BiDi ~ 0
-RESET_09
+COL_09
 Text GLabel 1900 2000 0    60   BiDi ~ 0
-RESET_10
+COL_10
 Text GLabel 1900 1800 0    60   BiDi ~ 0
-RESET_11
+COL_11
 Text GLabel 1900 2400 0    60   BiDi ~ 0
-RESET_12
+COL_12
 Wire Wire Line
 	1900 1800 2000 1800
@@
 Wire Wire Line
 	1900 3200 2000 3200
-NoConn ~ 2000 2500
-NoConn ~ 3100 2500
 Text GLabel 3200 2100 2    60   BiDi ~ 0
-SET_01
+COL_15
 Text GLabel 3200 2000 2    60   BiDi ~ 0
-SET_02
+COL_16
 Text GLabel 3200 1900 2    60   BiDi ~ 0
-SET_03
+COL_17
 Text GLabel 3200 1700 2    60   BiDi ~ 0
-SET_04
+COL_18
 Text GLabel 3200 2300 2    60   BiDi ~ 0
-SET_05
+COL_19
 Text GLabel 3200 1800 2    60   BiDi ~ 0
-SET_06
+COL_20
 Text GLabel 3200 2400 2    60   BiDi ~ 0
-SET_07
+COL_21
 Text GLabel 3200 3100 2    60   BiDi ~ 0
-SET_08
+COL_22
 Text GLabel 3200 3000 2    60   BiDi ~ 0
-SET_09
+COL_23
 Text GLabel 3200 2900 2    60   BiDi ~ 0
-SET_10
+COL_24
 Text GLabel 3200 2800 2    60   BiDi ~ 0
-SET_11
+COL_25
 Text GLabel 3200 2600 2    60   BiDi ~ 0
-SET_12
+COL_26
 Text GLabel 3200 2700 2    60   BiDi ~ 0
-SET_13
+COL_27
 Wire Wire Line
 	3100 3100 3200 3100
@@
 	1    0    0    -1
 $EndComp
+Text GLabel 1900 2500 0    60   BiDi ~ 0
+COL_14
+Wire Wire Line
+	1900 2500 2000 2500
 $Comp
 L FP2800a:FP2800A IC1
@@
 	1    0    0    -1
 $EndComp
+Text GLabel 3200 2500 2    60   BiDi ~ 0
+COL_28
+Wire Wire Line
+	3100 2500 3200 2500
 $EndSCHEMATC
